File: KiCad/Low-Pass-Filter-Board/Low-Pass-Filter-Board.kicad_pcb (KiCad board)
At the start: 2 copper layers, 49.3 x 16 mm, 15 parts, among them J1 Conn_01x03_Header, J2 Conn_01x03_Header

Commit message: live code changes during session
Connections:
- C1 pad 2: Net-(J1-Pin_1) -> GND
- C10 pad 2: Net-(J1-Pin_1) -> GND
- C2 pad 2: Net-(J1-Pin_1) -> GND
- C3 pad 2: Net-(J1-Pin_1) -> GND
- C4 pad 2: Net-(J1-Pin_1) -> GND
- C7 pad 2: Net-(J1-Pin_1) -> GND
- C8 pad 2: Net-(J1-Pin_1) -> GND
- C9 pad 2: Net-(J1-Pin_1) -> GND
- J1 pad 1: Net-(J1-Pin_1) -> GND
- J1 pad 3: Net-(J1-Pin_3) -> GND
- J2 pad 1: Net-(J1-Pin_1) -> GND
- J2 pad 3: Net-(J1-Pin_3) -> GND
Routing:
- net Net-(J1-Pin_1): track 52.4 -> 0.00 mm
- net Net-(J1-Pin_3): track 44.3 -> 0.00 mm
- added copper zone on F.Cu, net GND
Changed lines of the file:
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@@
   (net 0 "")
   (net 1 "Net-(J1-Pin_2)")
-  (net 2 "Net-(J1-Pin_1)")
+  (net 2 "GND")
   (net 3 "Net-(C3-Pad1)")
   (net 4 "Net-(C5-Pad2)")
   (net 5 "Net-(J2-Pin_2)")
-  (net 6 "Net-(J1-Pin_3)")
   (footprint "Capacitor_SMD:C_1206_3216Metric_Pad1.33x1.80mm_HandSolder" (layer "F.Cu")
     (at 132.0415 92.964)
@@
       (net 1 "Net-(J1-Pin_2)") (pintype "passive"))
     (pad "2" smd roundrect (at 1.5625 0 270) (size 1.325 1.8) (layers "F.Cu" "F.Paste" "F.Mask") (roundrect_rratio 0.1886792453)
-      (net 2 "Net-(J1-Pin_1)") (pintype "passive"))
+      (net 2 "GND") (pintype "passive"))
     (model "${KICAD6_3DMODEL_DIR}/Capacitor_SMD.3dshapes/C_1206_3216Metric.wrl"
       (offset (xyz 0 0 0))
@@
       (net 4 "Net-(C5-Pad2)") (pintype "passive"))
     (pad "2" smd roundrect (at 1.5625 0 270) (size 1.325 1.8) (layers "F.Cu" "F.Paste" "F.Mask") (roundrect_rratio 0.1886792453)
-      (net 2 "Net-(J1-Pin_1)") (pintype "passive"))
+      (net 2 "GND") (pintype "passive"))
     (model "${KICAD6_3DMODEL_DIR}/Capacitor_SMD.3dshapes/C_1206_3216Metric.wrl"
       (offset (xyz 0 0 0))
@@
       (net 5 "Net-(J2-Pin_2)") (pintype "passive"))
     (pad "2" smd roundrect (at 1.5625 0 270) (size 1.325 1.8) (layers "F.Cu" "F.Paste" "F.Mask") (roundrect_rratio 0.1886792453)
-      (net 2 "Net-(J1-Pin_1)") (pintype "passive"))
+      (net 2 "GND") (pintype "passive"))
     (model "${KICAD6_3DMODEL_DIR}/Capacitor_SMD.3dshapes/C_1206_3216Metric.wrl"
       (offset (xyz 0 0 0))
@@
       (net 1 "Net-(J1-Pin_2)") (pintype "passive"))
     (pad "2" smd roundrect (at 1.5625 0 270) (size 1.325 1.8) (layers "F.Cu" "F.Paste" "F.Mask") (roundrect_rratio 0.1886792453)
-      (net 2 "Net-(J1-Pin_1)") (pintype "passive"))
+      (net 2 "GND") (pintype "passive"))
     (model "${KICAD6_3DMODEL_DIR}/Capacitor_SMD.3dshapes/C_1206_3216Metric.wrl"
       (offset (xyz 0 0 0))
@@
       (net 5 "Net-(J2-Pin_2)") (pintype "passive"))
     (pad "2" smd roundrect (at 1.5625 0 270) (size 1.325 1.8) (layers "F.Cu" "F.Paste" "F.Mask") (roundrect_rratio 0.1886792453)
-      (net 2 "Net-(J1-Pin_1)") (pintype "passive"))
+      (net 2 "GND") (pintype "passive"))
     (model "${KICAD6_3DMODEL_DIR}/Capacitor_SMD.3dshapes/C_1206_3216Metric.wrl"
       (offset (xyz 0 0 0))
@@
       (net 3 "Net-(C3-Pad1)") (pintype "passive"))
     (pad "2" smd roundrect (at 1.5625 0 270) (size 1.325 1.8) (layers "F.Cu" "F.Paste" "F.Mask") (roundrect_rratio 0.1886792453)
-      (net 2 "Net-(J1-Pin_1)") (pintype "passive"))
+      (net 2 "GND") (pintype "passive"))
     (model "${KICAD6_3DMODEL_DIR}/Capacitor_SMD.3dshapes/C_1206_3216Metric.wrl"
       (offset (xyz 0 0 0))
@@
       (net 4 "Net-(C5-Pad2)") (pintype "passive"))
     (pad "2" smd roundrect (at 1.5625 0 270) (size 1.325 1.8) (layers "F.Cu" "F.Paste" "F.Mask") (roundrect_rratio 0.1886792453)
-      (net 2 "Net-(J1-Pin_1)") (pintype "passive"))
+      (net 2 "GND") (pintype "passive"))
     (model "${KICAD6_3DMODEL_DIR}/Capacitor_SMD.3dshapes/C_1206_3216Metric.wrl"
       (offset (xyz 0 0 0))
@@
       (net 3 "Net-(C3-Pad1)") (pintype "passive"))
     (pad "2" smd roundrect (at 1.5625 0 270) (size 1.325 1.8) (layers "F.Cu" "F.Paste" "F.Mask") (roundrect_rratio 0.1886792453)
-      (net 2 "Net-(J1-Pin_1)") (pintype "passive"))
+      (net 2 "GND") (pintype "passive"))
     (model "${KICAD6_3DMODEL_DIR}/Capacitor_SMD.3dshapes/C_1206_3216Metric.wrl"
       (offset (xyz 0 0 0))
@@
       (stroke (width 0.1) (type solid)) (layer "B.Fab"))
     (pad "1" thru_hole rect (at 0 0) (size 0.85 0.85) (drill 0.5) (layers "*.Cu" "*.Mask")
-      (net 2 "Net-(J1-Pin_1)") (pinfunction "Pin_1") (pintype "passive"))
+      (net 2 "GND") (pinfunction "Pin_1") (pintype "passive"))
     (pad "2" thru_hole oval (at 0 -1) (size 0.85 0.85) (drill 0.5) (layers "*.Cu" "*.Mask")
       (net 1 "Net-(J1-Pin_2)") (pinfunction "Pin_2") (pintype "passive"))
     (pad "3" thru_hole oval (at 0 -2) (size 0.85 0.85) (drill 0.5) (layers "*.Cu" "*.Mask")
-      (net 6 "Net-(J1-Pin_3)") (pinfunction "Pin_3") (pintype "passive"))
+      (net 2 "GND") (pinfunction "Pin_3") (pintype "passive"))
     (model "${KICAD6_3DMODEL_DIR}/Connector_PinHeader_1.00mm.3dshapes/PinHeader_1x03_P1.00mm_Vertical.wrl"
       (offset (xyz 0 0 0))
@@
       (stroke (width 0.1) (type solid)) (layer "B.Fab"))
     (pad "1" thru_hole rect (at 0 0) (size 0.85 0.85) (drill 0.5) (layers "*.Cu" "*.Mask")
-      (net 2 "Net-(J1-Pin_1)") (pinfunction "Pin_1") (pintype "passive"))
+      (net 2 "GND") (pinfunction "Pin_1") (pintype "passive"))
     (pad "2" thru_hole oval (at 0 -1) (size 0.85 0.85) (drill 0.5) (layers "*.Cu" "*.Mask")
       (net 5 "Net-(J2-Pin_2)") (pinfunction "Pin_2") (pintype "passive"))
     (pad "3" thru_hole oval (at 0 -2) (size 0.85 0.85) (drill 0.5) (layers "*.Cu" "*.Mask")
-      (net 6 "Net-(J1-Pin_3)") (pinfunction "Pin_3") (pintype "passive"))
+      (net 2 "GND") (pinfunction "Pin_3") (pintype "passive"))
     (model "${KICAD6_3DMODEL_DIR}/Connector_PinHeader_1.00mm.3dshapes/PinHeader_1x03_P1.00mm_Vertical.wrl"
       (offset (xyz 0 0 0))
@@
   (segment (start 119.276 96.52) (end 116.332 96.52) (width 0.25) (layer "F.Cu") (net 1))
   (segment (start 116.332 98.983) (end 116.332 96.52) (width 0.25) (layer "F.Cu") (net 1))
-  (segment (start 135.89 102.108) (end 139.7 102.108) (width 0.25) (layer "F.Cu") (net 2))
-  (segment (start 110.49 102.108) (end 112.522 102.108) (width 0.25) (layer "F.Cu") (net 2))
-  (segment (start 153.162 102.108) (end 151.13 102.108) (width 0.25) (layer "F.Cu") (net 2))
-  (segment (start 153.67 101.6) (end 153.162 102.108) (width 0.25) (layer "F.Cu") (net 2))
-  (segment (start 109.728 101.346) (end 109.728 97.52) (width 0.25) (layer "F.Cu") (net 2))
-  (segment (start 124.46 102.108) (end 116.332 102.108) (width 0.25) (layer "F.Cu") (net 2))
-  (segment (start 135.89 102.108) (end 128.27 102.108) (width 0.25) (layer "F.Cu") (net 2))
-  (segment (start 112.522 102.108) (end 115.062 102.108) (width 0.25) (layer "F.Cu") (net 2))
-  (segment (start 115.062 102.108) (end 116.332 102.108) (width 0.25) (layer "F.Cu") (net 2))
-  (segment (start 147.32 102.108) (end 151.13 102.108) (width 0.25) (layer "F.Cu") (net 2))
-  (segment (start 153.67 97.52) (end 153.67 101.6) (width 0.25) (layer "F.Cu") (net 2))
-  (segment (start 109.728 101.346) (end 110.49 102.108) (width 0.25) (layer "F.Cu") (net 2))
-  (segment (start 147.32 102.108) (end 139.7 102.108) (width 0.25) (layer "F.Cu") (net 2))
-  (segment (start 124.46 102.108) (end 128.27 102.108) (width 0.25) (layer "F.Cu") (net 2))
   (segment (start 130.5175 90.17) (end 130.302 90.17) (width 0.25) (layer "F.Cu") (net 3))
   (segment (start 124.46 96.52) (end 126.492 96.52) (width 0.25) (layer "F.Cu") (net 3))
@@
   (segment (start 151.13 98.983) (end 151.13 96.52) (width 0.25) (layer "F.Cu") (net 5))
   (segment (start 147.32 96.52) (end 149.352 96.52) (width 0.25) (layer "F.Cu") (net 5))
-  (segment (start 153.245001 95.095001) (end 110.152999 95.095001) (width 0.25) (layer "B.Cu") (net 6))
-  (segment (start 153.67 95.52) (end 153.245001 95.095001) (width 0.25) (layer "B.Cu") (net 6))
-  (segment (start 110.152999 95.095001) (end 109.728 95.52) (width 0.25) (layer "B.Cu") (net 6))
+  (zone (net 2) (net_name "GND") (layer "F.Cu") (name "GND") (hatch edge 0.5)
+    (connect_pads (clearance 0.5))
+    (min_thickness 0.25) (filled_areas_thickness no)
+    (fill yes (thermal_gap 0.5) (thermal_bridge_width 0.5))
+    (polygon
+      (pts
+        (xy 157.48 104.902)
+        (xy 157.48 87.376)
+        (xy 106.426 87.376)
+        (xy 106.426 104.902)
+      )
+    )
+  )
   (group "" (id dadc619e-4783-41d8-9074-2524729f2a4f)
     (members
