File: KiCad/Low-Pass-Filter-Board/Low-Pass-Filter-Board.kicad_sch (KiCad schematic)
At the start: 15 parts, among them J1 Conn_01x03_Header, J2 Conn_01x03_Header

Commit message: live code changes during session
Connections:
- net GND: now reaches C1.2, C10.2, C2.2, C3.2, C4.2, C7.2, C8.2, C9.2, J1.1 (Pin_1), J2.1 (Pin_1)
- net GND: now also J1.3 (Pin_3), J2.3 (Pin_3)
