File: KiCad/Presentation-Schematics/Session2/Session10/Session10/Session10.kicad_sch (KiCad schematic)
At the start: 4 parts, among them U1 ESP32-WROOM-32

Commit message: updated schematic
Parts:
- added BRD3-DS1307: ~, Connector_PinHeader_2.54mm:PinHeader_1x05_P2.54mm_Vertical, symbol ILoveHamRadio:DS1307_RTC_BRD
- added BRD4-GPS: ~, Connector_PinHeader_2.54mm:PinHeader_1x05_P2.54mm_Vertical, symbol ILoveHamRadio:NEO-6M_BRD
- BRD1-SI5351A: renamed from U2; footprint (none) -> Connector_PinHeader_2.54mm:PinHeader_1x07_P2.54mm_Vertical
- Brd2-SSD1306-OLED: renamed from Brd1; footprint (none) -> Connector_PinHeader_2.54mm:PinHeader_1x04_P2.54mm_Vertical
- Encoder1: renamed from SW1; footprint (none) -> Connector_PinHeader_2.54mm:PinHeader_1x05_P2.54mm_Vertical
Connections:
- net +3.3V: now also BRD3-DS1307.4 (VCC), BRD4-GPS.5 (VCC)
- net GND: now also BRD3-DS1307.5 (GND), BRD4-GPS.4 (GND)
- net at Encoder1.3 (SW): now also U1.31 (IO19); no longer U1.19 (SCS/CMD)
- net at Encoder1.4 (DT): now also U1.30 (IO18); no longer U1.18 (SWP/SD3)
- net at BRD1-SI5351A.4 (SCL), Brd2-SSD1306-OLED.3 (SCL), U1.22 (SDI/SD1): now also BRD3-DS1307.2 (SCL)
- net at BRD1-SI5351A.3 (SDA), Brd2-SSD1306-OLED.4 (SDA), U1.21 (SDO/SD0): now also BRD3-DS1307.3 (SDA)
- net at U1.27 (IO16): now also BRD4-GPS.2 (TXD)
- net at U1.28 (IO17): now also BRD4-GPS.3 (RXD)
Other:
- moved on the sheet: Brd2-SSD1306-OLED, U1
